File: hardware/pcb/pcb.kicad_sch (KiCad schematic)
At the start: 49 parts, among them CN101 XT30PW-M, U101 RP2040, U102 W25Q128JVP, U103 ICM-42688-P, U104 MIC5219-3.3YM5, U105 MIC5219-3.3YM5, U106 AMS1117-5.0, U107 S4B-XH-SM4-TB-, Y101 12MHz

Commit message: redesign
Parts:
- added H101, H102, H103, H104: MountingHole, MountingHole:MountingHole_3.2mm_M3_DIN965, symbol Mechanical:MountingHole
- added TP101: SWCLK, TestPoint:TestPoint_Pad_D1.0mm, symbol Connector:TestPoint
- added TP102: SWD, TestPoint:TestPoint_Pad_D1.0mm, symbol Connector:TestPoint
Connections:
- net SWCLK: now also TP101.1
- net SWD: now also TP102.1
Other:
- moved on the sheet: C103, C126, C127, Card101, R102, R104, R105, R106, R107, R108, R109, U102
